File: Hardware/rpi/external/RP2040/Multiplexed_PMP/Multiplexed_PMP.brd (EAGLE design)
At the start: 80 x 77.5 mm, 19 parts, among them IC1 74HC245D, IC2 74HC245D, IC3 74HC245D, IC4 74HC245D, IC5 74LS245DW, J1 RASPBERRYPI-40-PIN-GPIO_PTH_N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

Commit message: Add files via upload
Parts:
- moved J1 48.3 mm to (5.08, 26.7), turned to 90 degrees
Routing:
- net DAT6: track 143.9 -> 61.6 mm, vias 0 -> 4
- net DAT5: track 114.2 -> 62.3 mm, vias 3 -> 4
- net GND: track 548.8 -> 509.3 mm, vias 4 -> 0
- net DAT_D5: track 78.6 -> 49.7 mm, vias 0 -> 1
- net RESET: track 27.3 -> 55.4 mm, vias 0 -> 1
- net WR2: track 43.9 -> 20.1 mm, vias 1 -> 0
- net DAT1: track 105.0 -> 81.4 mm, vias 3 -> 4
- net DAT7: track 87.8 -> 109.2 mm
- net DAT2: track 96.1 -> 76.8 mm, vias 3 -> 5
- net DAT_B0: track 80.0 -> 63.8 mm
- net WR3: track 14.6 -> 30.0 mm, vias 0 -> 1
- net DAT_B1: track 74.6 -> 60.0 mm
- net VCC: track 158.7 -> 172.4 mm
- net WR1: track 22.0 -> 30.9 mm, vias 1 -> 0
- net DAT_C1: track 79.5 -> 71.7 mm
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